File: pcb/kicad/LED_MATRIX_ARRAY_1.kicad_sch (KiCad schematic)
At the start: 128 parts

Commit message: Update parts/mpns/descriptions etc.
- Incorrect LED part, was 0805 package instead of 0603
- Added MPNs for other parts (mostly ones I already own multiples of)
- Update schematics?
Parts:
- D101, D102, D103, D104, D105, D106, D107, D108, D109, D110, D111, D112, D113, D114, D115, D116, D201, D202, D203, D204, D205, D206, D207, D208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: value LTST-C171KRKT -> LTST-C190KRKT; MPN LTST-C171KRKT -> LTST-C190KRKT
