File: pcb/kicad/LED_MATRIX_ARRAY_2.kicad_sch (KiCad schematic)
At the start: 128 parts

Commit message: Update bom/mpn attributes
Parts:
- D117, D118, D119, D120, D121, D122, D123, D124, D125, D126, D127, D128, D129, D130, D131, D132, D217, D218, D219, D220, D221, D222, D223, D224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: value LTST-C190KRKT -> LED Matrix (RED)
