File: pcb/kicad/STM32_MCU.kicad_sch (KiCad schematic)
At the start: 13 parts, among them J2 Conn_ARM_JTAG_SWD_10, SW1 SW_Push, U2 STM32G431K8Tx

Commit message: Update parts/mpns/descriptions etc.
- Incorrect LED part, was 0805 package instead of 0603
- Added MPNs for other parts (mostly ones I already own multiples of)
- Update schematics?
Parts:
- D3: footprint Diode_SMD:Nexperia_DSN1608-2_1.6x0.8mm -> Diode_SMD:D_SOD-523; MPN (none) -> PESD5V0X1UAB,115
- R4: MPN (none) -> RT0603DRE071KL
Changed lines of the file:
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@@
 			)
 		)
-		(property "Footprint" "Diode_SMD:Nexperia_DSN1608-2_1.6x0.8mm"
+		(property "Footprint" "Diode_SMD:D_SOD-523"
 			(at 83.185 57.15 0)
 			(effects
@@
 			)
 		)
-		(property "Datasheet" "https://assets.nexperia.com/documents/data-sheet/PTVS5V0Z1USKP.pdf"
+		(property "Datasheet" ""
 			(at 87.63 57.15 0)
 			(effects
@@
 			)
 		)
-		(property "Description" "5V, 2000W TVS unidirectional diode, DSN1608-2"
+		(property "Description" "5V, TVS unidirectional diode"
 			(at 87.63 57.15 0)
+			(effects
+				(font
+					(size 1.27 1.27)
+				)
+				(hide yes)
+			)
+		)
+		(property "MPN" "PESD5V0X1UAB,115"
+			(at 87.63 57.15 90)
 			(effects
 				(font
@@
 			(at 167.64 101.6 0)
 			(effects
+				(font
+					(size 1.27 1.27)
+				)
+				(hide yes)
+			)
+		)
+		(property "MPN" "RT0603DRE071KL"
+			(at 167.64 101.6 0)
+			(effects

Commit message: Update capcitor annotations
- One less capacitor therefore the symbol annotations need to be changed
Parts:
- renumbered C11 to C10, C12 to C11, C13 to C12, C10 to C7
Changed lines of the file:
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@@
 	(title_block
 		(title "STM32G431Kx Schematic")
-		(date "2025-05-06")
-		(rev "v05")
+		(date "2025-05-21")
+		(rev "v06")
 		(comment 1 "No ADC therefore tying VDDA to VDD and GNDA to GND")
 		(comment 2 "Decoupling capacitor info can be found on datasheet and application note AN5093 ")
@@
 		(on_board yes)
 		(dnp no)
-		(property "Reference" "C11"
+		(property "Reference" "C10"
 			(at 80.01 149.86 0)
 			(effects
@@
 			(project "i2s_spekky_matrix"
 				(path "/e164be4c-4870-49b4-a08f-d162a756edc1/a94a638a-4aca-4eb4-a11b-127bd621569f"
-					(reference "C11")
+					(reference "C10")
 					(unit 1)
 				)
@@
 		(on_board yes)
 		(dnp no)
-		(property "Reference" "C13"
+		(property "Reference" "C12"
 			(at 113.03 149.86 0)
 			(effects
@@
 			(project "i2s_spekky_matrix"
 				(path "/e164be4c-4870-49b4-a08f-d162a756edc1/a94a638a-4aca-4eb4-a11b-127bd621569f"
-					(reference "C13")
+					(reference "C12")
 					(unit 1)
 				)
@@
 		(on_board yes)
 		(dnp no)
-		(property "Reference" "C12"
+		(property "Reference" "C11"
 			(at 101.6 149.86 0)
 			(effects
@@
 			(project "i2s_spekky_matrix"
 				(path "/e164be4c-4870-49b4-a08f-d162a756edc1/a94a638a-4aca-4eb4-a11b-127bd621569f"
-					(reference "C12")
+					(reference "C11")
 					(unit 1)
 				)
@@
 		(on_board yes)
 		(dnp no)
-		(property "Reference" "C10"
+		(property "Reference" "C7"
 			(at 72.39 55.88 0)
 			(effects
@@
 			(project ""
 				(path "/e164be4c-4870-49b4-a08f-d162a756edc1/a94a638a-4aca-4eb4-a11b-127bd621569f"
-					(reference "C10")
+					(reference "C7")
 					(unit 1)
 				)

Commit message: Add comment for pb3 (spi_clk/swo)
- PB3 is being used for SPI_CLK
- However is also connected to SWO, the programmer can choose to enable
  SWO at the cost of losing SPI_CLK (maybe useful for debug stages)
Other:
- note added: "PB3 cannot be used for both SPI_CLK and SWO Programmer must configure between them Spekky matrix doesn't use SWO"
Changed lines of the file:
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@@
 	(title_block
 		(title "STM32G431Kx Schematic")
-		(date "2025-05-21")
-		(rev "v06")
+		(date "2025-05-22")
+		(rev "v07")
 		(comment 1 "No ADC therefore tying VDDA to VDD and GNDA to GND")
 		(comment 2 "Decoupling capacitor info can be found on datasheet and application note AN5093 ")
@@
 		(effects
 			(font
+				(size 1.27 1.27)
+			)
+			(justify left)
+		)
+	)
+	(text "PB3 cannot be used for both SPI_CLK and SWO\nProgrammer must configure between them\nSpekky matrix doesn't use SWO"
+		(exclude_from_sim no)
+		(at 28.702 89.408 0)
+		(effects
+			(font

Commit message: Add stm32 nrst comment
- Added a comment to inidicate the recommneded circuitry for the NRST
  pin as indicated in the STM32G4x datasheet
- This circuitry is also in the Nucleo line of devices (with the
  additional ESD protection), so the circuit should function
  without any issues
Other:
- note added: "Recommended external reset circuit: via DS12589 Rev 6 (STM32G4x datasheet) (plus additional ESD protection)"
Changed lines of the file:
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@@
 		(title "STM32G431Kx Schematic")
 		(date "2025-05-22")
-		(rev "v07")
+		(rev "v08")
 		(comment 1 "No ADC therefore tying VDDA to VDD and GNDA to GND")
 		(comment 2 "Decoupling capacitor info can be found on datasheet and application note AN5093 ")
@@
 		)
 	)
+	(text "Recommended external reset circuit:\nvia DS12589 Rev 6 (STM32G4x datasheet)\n(plus additional ESD protection)"
+		(exclude_from_sim no)
+		(at 59.436 36.576 0)
+		(effects
+			(font
+				(size 1.27 1.27)
+			)
+			(justify left)
+		)
+	)
