File: pcb/kicad/spekky_matrix.kicad_sch (KiCad schematic)
At the start: 4 parts

Commit message: Update gndref net to gnd
- Changes applied to schematic and PCB
- Using GNDREF symbol for GND but need to change the net name
Connections:
- net GNDREF renamed GND
Changed lines of the file:
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@@
 	(title_block
 		(title "Spekky Matrix Schematic")
-		(date "2025-05-22")
-		(rev "v20")
+		(date "2025-06-14")
+		(rev "v21")
 	)
 	(junction
@@
 		(on_board yes)
 		(dnp no)
-		(fields_autoplaced yes)
-		(property "Reference" "#PWR0119"
+		(property "Reference" "#PWR01"
 			(at 53.34 132.08 0)
 			(effects
@@
 			)
 		)
-		(property "Value" "GNDREF"
-			(at 53.34 130.81 0)
+		(property "Value" "GND"
+			(at 53.34 129.54 0)
 			(effects
 				(font
@@
 			)
 		)
-		(property "Description" "Power symbol creates a global label with name \"GNDREF\" , reference supply ground"
+		(property "Description" "Power symbol creates a global label with name \"GND\" , reference supply ground"
 			(at 53.34 125.73 0)
 			(effects
@@
 		)
 		(instances
-			(project ""
+			(project "spekky_matrix"
 				(path "/e164be4c-4870-49b4-a08f-d162a756edc1"
-					(reference "#PWR0119")
+					(reference "#PWR01")
 					(unit 1)
 				)
