File: pcb/kicad/spekky_matrix.kicad_sch (KiCad schematic)
At the start: 4 parts

Commit message: Correct stm32 outputs for led driver ic
- SPI CS is analogous to LE, but was instead mapped to OE which in my
  initial tests were tied to GND (all LEDs could be driven)
- Now SPI CS has been renamed to OE and is still mapped to OE pin on the
  STP led driver IC
- GPIO LE is now correctly mapped the LE input on the STP too
Other:
- sheet LED DRIVING ports: added GLOBAL_LED_OE; removed SPI_OE
- sheet STM32 MCU ports: added GPIO_OE, GPIO_SPI_CS; removed GPIO_LE, SPI_CS
Changed lines of the file:
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@@
 	(title_block
 		(title "Spekky Matrix Schematic")
-		(date "2025-06-29")
-		(rev "v24")
+		(date "2025-11-01")
+		(rev "v25")
 	)
 	(junction
@@
 			)
 		)
-		(pin "SPI_OE" input
-			(at 124.46 74.93 180)
-			(effects
-				(font
-					(size 1.27 1.27)
-				)
-				(justify left)
-			)
-		)
 		(pin "GPIO_LE" input
 			(at 124.46 77.47 180)
+			(effects
+				(font
+					(size 1.27 1.27)
+				)
+				(justify left)
+			)
+		)
+		(pin "GLOBAL_LED_OE" input
+			(at 124.46 74.93 180)
 			(effects
 				(font
@@
 			)
 		)
-		(pin "SPI_CS" output
-			(at 115.57 74.93 0)
-			(effects
-				(font
-					(size 1.27 1.27)
-				)
-				(justify right)
-			)
-		)
 		(pin "I2S_WS" output
 			(at 77.47 74.93 180)
@@
 			)
 		)
-		(pin "GPIO_LE" output
+		(pin "GPIO_OE" output
+			(at 115.57 74.93 0)
+			(effects
+				(font
+					(size 1.27 1.27)
+				)
+				(justify right)
+			)
+		)
+		(pin "GPIO_SPI_CS" output
 			(at 115.57 77.47 0)
 			(effects
