File: pcb/kicad/LED_DRIVING.kicad_sch (KiCad schematic)
At the start: 43 parts, among them Q1 DMP3125L-7, Q2 DMP3125L-7, Q3 DMP3125L-7, Q4 DMP3125L-7, Q5 DMP3125L-7, Q6 DMP3125L-7, Q7 DMP3125L-7, Q8 DMP3125L-7, U3 STP16CP05XT, U4 STP16CP05XT, U5 STP16CP05XT

Commit message: Add test points to schematic and pcb
- Test points are in the form of a 0402 (Imperial) diode footprint with
  pin 1 denoting the signal being tested and pin 2 always being GND
- Therefore the silkscreen GND has been omitted, follow the signal name
  to the "." which denotes pin 1
- 0402 package is intended for a oscilloscope probe with the ground
  probe tip for a low impedance path to ground
- ARM SWD test points can be via the hook clip along with a clip to
  ground nearby, as the SWD is a THT footprint I didn't feel the need to
  again expose out more pins for a SMD based test point
- Since the pads for the I2S mic are already exposed, it seemed
  counterintuitive to then make additional test points for the I2S
  pads. The silkscreen describes the pinout such that on-the-fly test
  points can be used in conjunction with nearby ground vias and pads
Parts:
- added TP10, TP11, TP12, TP13, TP14, TP15, TP16, TP17, TP18, TP19, TP20, TP21, TP22, TP23, TP24, TP25, TP26, TP27, TP28, TP29, TP30, TP31, TP32, TP33, TP34, TP35, TP36, TP37, TP38, TP39, TP4, TP40, TP41, TP42, TP43, TP44, TP45, TP46, TP47, TP48, TP49, TP5, TP50, TP51, TP52, TP53, TP54, TP55, TP6, TP7, TP8, TP9: TestPoint_2Pole, Diode_SMD:D_0402_1005Metric, symbol Connector:TestPoint_2Pole
Connections:
- net COL1: now also TP24.1
- net COL10: now also TP33.1
- net COL11: now also TP34.1
- net COL12: now also TP35.1
- net COL13: now also TP36.1
- net COL14: now also TP37.1
- net COL15: now also TP38.1
- net COL16: now also TP39.1
- net COL17: now also TP40.1
- net COL18: now also TP41.1
- net COL19: now also TP42.1
- net COL2: now also TP25.1
- net COL20: now also TP43.1
- net COL21: now also TP44.1
- net COL22: now also TP45.1
- net COL23: now also TP46.1
- net COL24: now also TP47.1
- net COL25: now also TP48.1
- net COL26: now also TP49.1
- net COL27: now also TP50.1
- net COL28: now also TP51.1
- net COL29: now also TP52.1
- net COL3: now also TP26.1
- net COL30: now also TP53.1
- net COL31: now also TP54.1
- net COL32: now also TP55.1
- net COL4: now also TP27.1
- net COL5: now also TP28.1
- net COL6: now also TP29.1
- net COL7: now also TP30.1
- net COL8: now also TP31.1
- net COL9: now also TP32.1
- net GND: now also TP10.2, TP11.2, TP12.2, TP13.2, TP14.2, TP15.2, TP16.2, TP17.2, TP18.2, TP19.2, TP20.2, TP21.2, TP22.2, TP23.2, TP24.2, TP25.2, TP26.2, TP27.2, TP28.2, TP29.2, TP30.2, TP31.2, TP32.2, TP33.2, TP34.2, TP35.2, TP36.2, TP37.2, TP38.2, TP39.2, TP4.2, TP40.2, TP41.2, TP42.2, TP43.2, TP44.2, TP45.2, TP46.2, TP47.2, TP48.2, TP49.2, TP5.2, TP50.2, TP51.2, TP52.2, TP53.2, TP54.2, TP55.2, TP6.2, TP7.2, TP8.2, TP9.2
- net GPIO_LE: now also TP13.1, TP16.1, TP19.1
- net ROW1: now also TP11.1
- net ROW2: now also TP10.1
- net ROW3: now also TP9.1
- net ROW4: now also TP8.1
- net ROW5: now also TP7.1
- net ROW6: now also TP6.1
- net ROW7: now also TP5.1
- net ROW8: now also TP4.1
- net SPI_CLK: now also TP14.1, TP17.1, TP20.1
- net SPI_MOSI: now also TP21.1
- net SPI_OE: now also TP12.1, TP15.1, TP18.1
- net SDO_CASCADE2: now reaches U3.2 (SDI), U4.22 (SDO)
- net SDO_CASCADE2: now also TP23.1
- net SDO_CASCADE1: now reaches U4.2 (SDI), U5.22 (SDO)
- net SDO_CASCADE1: now also TP22.1

Commit message: Update bom/mpn attributes
Parts:
- C13, C14, C15: MPN (none) -> C0603C104J3RACTU
- JP1, TP10, TP11, TP12, TP13, TP14, TP15, TP16, TP17, TP18, TP19, TP20, TP21, TP22, TP23, TP24, TP25, TP26, TP27, TP28, TP29, TP30, TP31, TP32, TP33, TP34, TP35, TP36, TP37, TP38, TP39, TP4, TP40, TP41, TP42, TP43, TP44, TP45, TP46, TP47, TP48, TP49, TP5, TP50, TP51, TP52, TP53, TP54, TP55, TP6, TP7, TP8, TP9: now left out of the parts list
Changed lines of the file:
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@@
 		(unit 1)
 		(exclude_from_sim no)
-		(in_bom yes)
+		(in_bom no)
 		(on_board yes)
 		(dnp no)
@@
 		(unit 1)
 		(exclude_from_sim no)
-		(in_bom yes)
+		(in_bom no)
 		(on_board yes)
 		(dnp no)
@@
 		(unit 1)
 		(exclude_from_sim no)
-		(in_bom yes)
+		(in_bom no)
 		(on_board yes)
 		(dnp no)
@@
 		(unit 1)
 		(exclude_from_sim no)
-		(in_bom yes)
+		(in_bom no)
 		(on_board yes)
 		(dnp no)
@@
 			)
 		)
+		(property "MPN" "C0603C104J3RACTU"
+			(at 345.44 78.74 0)
+			(effects
+				(font
+					(size 1.27 1.27)
+				)
+				(hide yes)
+			)
+		)
 		(pin "2"
 		)
@@
 		(unit 1)
 		(exclude_from_sim no)
-		(in_bom yes)
+		(in_bom no)
 		(on_board yes)
 		(dnp no)
@@
 		(unit 1)
 		(exclude_from_sim no)
-		(in_bom yes)
+		(in_bom no)
 		(on_board yes)
 		(dnp no)
@@
 		(unit 1)
 		(exclude_from_sim no)
-		(in_bom yes)
+		(in_bom no)
 		(on_board yes)
 		(dnp no)
@@
 		(unit 1)
 		(exclude_from_sim no)
-		(in_bom yes)
+		(in_bom no)
 		(on_board yes)
 		(dnp no)
@@
 		(unit 1)
 		(exclude_from_sim no)
-		(in_bom yes)
+		(in_bom no)
 		(on_board yes)
 		(dnp no)
@@
 		(unit 1)
 		(exclude_from_sim no)
-		(in_bom yes)
+		(in_bom no)
 		(on_board yes)
 		(dnp no)
@@
 		(unit 1)
 		(exclude_from_sim no)
-		(in_bom yes)
+		(in_bom no)
 		(on_board yes)
 		(dnp no)
@@
 		(unit 1)
 		(exclude_from_sim no)
-		(in_bom yes)
+		(in_bom no)
 		(on_board yes)
 		(dnp no)
@@
 		(unit 1)
 		(exclude_from_sim no)
-		(in_bom yes)
+		(in_bom no)
 		(on_board yes)
 		(dnp no)
@@
 		(unit 1)
 		(exclude_from_sim no)
-		(in_bom yes)
+		(in_bom no)
 		(on_board yes)
 		(dnp no)
@@
 			)
 		)
+		(property "MPN" "C0603C104J3RACTU"
+			(at 146.05 77.47 0)
+			(effects
+				(font
+					(size 1.27 1.27)
+				)
+				(hide yes)
+			)
+		)
 		(pin "2"
 		)
@@
 		(unit 1)
 		(exclude_from_sim no)
-		(in_bom yes)
+		(in_bom no)
 		(on_board yes)
 		(dnp no)
@@
 		(unit 1)
 		(exclude_from_sim no)
-		(in_bom yes)
+		(in_bom no)
 		(on_board yes)
 		(dnp no)
@@
 		(unit 1)
 		(exclude_from_sim no)
-		(in_bom yes)
+		(in_bom no)
 		(on_board yes)
 		(dnp no)
@@
 		(unit 1)
 		(exclude_from_sim no)
-		(in_bom yes)
+		(in_bom no)
 		(on_board yes)
 		(dnp no)
@@
 		(unit 1)
 		(exclude_from_sim no)
-		(in_bom yes)
+		(in_bom no)
 		(on_board yes)
 		(dnp no)
@@
 		(unit 1)
 		(exclude_from_sim yes)
-		(in_bom yes)
+		(in_bom no)
 		(on_board yes)
 		(dnp no)
@@
 		(unit 1)
 		(exclude_from_sim no)
-		(in_bom yes)
+		(in_bom no)
 		(on_board yes)
 		(dnp no)
@@
 		(unit 1)
 		(exclude_from_sim no)
-		(in_bom yes)
+		(in_bom no)
 		(on_board yes)
 		(dnp no)
@@
 		(unit 1)
 		(exclude_from_sim no)
-		(in_bom yes)
+		(in_bom no)
 		(on_board yes)
 		(dnp no)
@@
 		(unit 1)
 		(exclude_from_sim no)
-		(in_bom yes)
+		(in_bom no)
 		(on_board yes)
 		(dnp no)
@@
 		(unit 1)
 		(exclude_from_sim no)
-		(in_bom yes)
+		(in_bom no)
 		(on_board yes)
 		(dnp no)
@@
 		(unit 1)
 		(exclude_from_sim no)
-		(in_bom yes)
+		(in_bom no)
 		(on_board yes)
 		(dnp no)
@@
 		(unit 1)
 		(exclude_from_sim no)
-		(in_bom yes)
+		(in_bom no)
 		(on_board yes)
 		(dnp no)
@@
 		(unit 1)
 		(exclude_from_sim no)
-		(in_bom yes)
+		(in_bom no)
 		(on_board yes)
 		(dnp no)
@@
 		(unit 1)
 		(exclude_from_sim no)
-		(in_bom yes)
+		(in_bom no)
 		(on_board yes)
 		(dnp no)
@@
 		(unit 1)
 		(exclude_from_sim no)
-		(in_bom yes)
+		(in_bom no)
 		(on_board yes)
 		(dnp no)
@@
 		(unit 1)
 		(exclude_from_sim no)
-		(in_bom yes)
+		(in_bom no)
 		(on_board yes)
 		(dnp no)
@@
 			)
 		)
+		(property "MPN" "C0603C104J3RACTU"
+			(at 247.65 78.74 0)
+			(effects
+				(font
+					(size 1.27 1.27)
+				)
+				(hide yes)
+			)
+		)
 		(pin "2"
 		)
@@
 		(unit 1)
 		(exclude_from_sim no)
-		(in_bom yes)
+		(in_bom no)
 		(on_board yes)
 		(dnp no)
@@
 		(unit 1)
 		(exclude_from_sim no)
-		(in_bom yes)
+		(in_bom no)
 		(on_board yes)
 		(dnp no)
@@
 		(unit 1)
 		(exclude_from_sim no)
-		(in_bom yes)
+		(in_bom no)
 		(on_board yes)
 		(dnp no)
@@
 		(unit 1)
 		(exclude_from_sim no)
-		(in_bom yes)
+		(in_bom no)
 		(on_board yes)
 		(dnp no)
@@
 		(unit 1)
 		(exclude_from_sim no)
-		(in_bom yes)
+		(in_bom no)
 		(on_board yes)
 		(dnp no)
@@
 		(unit 1)
 		(exclude_from_sim no)
-		(in_bom yes)
+		(in_bom no)
 		(on_board yes)
 		(dnp no)
@@
 		(unit 1)
 		(exclude_from_sim no)
-		(in_bom yes)
+		(in_bom no)
 		(on_board yes)
 		(dnp no)
@@
 		(unit 1)
 		(exclude_from_sim no)
-		(in_bom yes)
+		(in_bom no)
 		(on_board yes)
 		(dnp no)
@@
 		(unit 1)
 		(exclude_from_sim no)
-		(in_bom yes)
+		(in_bom no)
 		(on_board yes)
 		(dnp no)
@@
 		(unit 1)
 		(exclude_from_sim no)
-		(in_bom yes)
+		(in_bom no)
 		(on_board yes)
 		(dnp no)
@@
 		(unit 1)
 		(exclude_from_sim no)
-		(in_bom yes)
+		(in_bom no)
 		(on_board yes)
 		(dnp no)
@@
 		(unit 1)
 		(exclude_from_sim no)
-		(in_bom yes)
+		(in_bom no)
 		(on_board yes)
 		(dnp no)
@@
 		(unit 1)
 		(exclude_from_sim no)
-		(in_bom yes)
+		(in_bom no)
 		(on_board yes)
 		(dnp no)
@@
 		(unit 1)
 		(exclude_from_sim no)
-		(in_bom yes)
+		(in_bom no)
 		(on_board yes)
 		(dnp no)
@@
 		(unit 1)
 		(exclude_from_sim no)
-		(in_bom yes)
+		(in_bom no)
 		(on_board yes)
 		(dnp no)
@@
 		(unit 1)
 		(exclude_from_sim no)
-		(in_bom yes)
+		(in_bom no)
 		(on_board yes)
 		(dnp no)
@@
 		(unit 1)
 		(exclude_from_sim no)
-		(in_bom yes)
+		(in_bom no)
 		(on_board yes)
 		(dnp no)
@@
 		(unit 1)
 		(exclude_from_sim no)
-		(in_bom yes)
+		(in_bom no)
 		(on_board yes)
 		(dnp no)
@@
 		(unit 1)
 		(exclude_from_sim no)
-		(in_bom yes)
+		(in_bom no)
 		(on_board yes)
 		(dnp no)
@@
 		(unit 1)
 		(exclude_from_sim no)
-		(in_bom yes)
+		(in_bom no)
 		(on_board yes)
 		(dnp no)
@@
 		(unit 1)
 		(exclude_from_sim no)
-		(in_bom yes)
+		(in_bom no)
 		(on_board yes)
 		(dnp no)
@@
 		(unit 1)
 		(exclude_from_sim no)
-		(in_bom yes)
+		(in_bom no)
 		(on_board yes)
 		(dnp no)

Commit message: Correct stm32 outputs for led driver ic
- SPI CS is analogous to LE, but was instead mapped to OE which in my
  initial tests were tied to GND (all LEDs could be driven)
- Now SPI CS has been renamed to OE and is still mapped to OE pin on the
  STP led driver IC
- GPIO LE is now correctly mapped the LE input on the STP too
Connections:
- net SPI_OE renamed GLOBAL_LED_OE
Changed lines of the file:
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@@
 	(title_block
 		(title "8x32 LED Matrix")
-		(date "2025-06-27")
-		(rev "v07")
+		(date "2025-11-01")
+		(rev "v08")
 		(comment 4 "STP16CP05 based cascaded LED matrices")
 	)
@@
 		)
 	)
-	(hierarchical_label "SPI_OE"
+	(hierarchical_label "GLOBAL_LED_OE"
 		(shape input)
 		(at 325.12 87.63 270)
@@
 		)
 	)
-	(hierarchical_label "SPI_OE"
+	(hierarchical_label "GLOBAL_LED_OE"
 		(shape input)
 		(at 227.33 87.63 270)
@@
 		)
 	)
-	(hierarchical_label "SPI_OE"
+	(hierarchical_label "GLOBAL_LED_OE"
 		(shape input)
 		(at 365.76 177.8 180)
@@
 		)
 	)
-	(hierarchical_label "SPI_OE"
+	(hierarchical_label "GLOBAL_LED_OE"
 		(shape input)
 		(at 365.76 187.96 180)
@@
 		)
 	)
-	(hierarchical_label "SPI_OE"
+	(hierarchical_label "GLOBAL_LED_OE"
 		(shape input)
 		(at 365.76 167.64 180)
@@
 		)
 	)
-	(hierarchical_label "SPI_OE"
+	(hierarchical_label "GLOBAL_LED_OE"
 		(shape input)
 		(at 127 86.36 270)

Commit message: Replace test point footprints
- Quite difficult to probe the 0402 SMD sized test points with my PCBite
  probes
- End up scraping up the PCB trying to probe my test points as the gap
  is too small (on the 0402 footprint)
- The 0805 and microMELF footprints are appropriately sized for hands
  free probing
- Used microMELF footprints where space was very tight (as the microMELF
  occupies a slightly smaller area)
Parts:
- TP10, TP12, TP13, TP14, TP15, TP17, TP18, TP19, TP20, TP21, TP22, TP23, TP6, TP7, TP8, TP9: footprint Diode_SMD:D_0402_1005Metric -> Diode_SMD:D_MicroMELF
- TP11, TP16, TP24, TP25, TP26, TP27, TP28, TP29, TP30, TP31, TP32, TP33, TP34, TP35, TP36, TP37, TP38, TP39, TP4, TP40, TP41, TP42, TP43, TP44, TP45, TP46, TP47, TP48, TP49, TP5, TP50, TP51, TP52, TP53, TP54, TP55: footprint Diode_SMD:D_0402_1005Metric -> Diode_SMD:D_0805_2012Metric
Changed lines of the file:
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@@
 			)
 		)
-		(property "Footprint" "Diode_SMD:D_0402_1005Metric"
+		(property "Footprint" "Diode_SMD:D_0805_2012Metric"
 			(at 397.51 107.95 0)
 			(effects
@@
 			)
 		)
-		(property "Footprint" "Diode_SMD:D_0402_1005Metric"
+		(property "Footprint" "Diode_SMD:D_MicroMELF"
 			(at 369.57 146.05 0)
 			(effects
@@
 			)
 		)
-		(property "Footprint" "Diode_SMD:D_0402_1005Metric"
+		(property "Footprint" "Diode_SMD:D_0805_2012Metric"
 			(at 397.51 179.07 0)
 			(effects
@@
 			)
 		)
-		(property "Footprint" "Diode_SMD:D_0402_1005Metric"
+		(property "Footprint" "Diode_SMD:D_MicroMELF"
 			(at 370.84 190.5 0)
 			(effects
@@
 			)
 		)
-		(property "Footprint" "Diode_SMD:D_0402_1005Metric"
+		(property "Footprint" "Diode_SMD:D_0805_2012Metric"
 			(at 397.51 123.19 0)
 			(effects
@@
 			)
 		)
-		(property "Footprint" "Diode_SMD:D_0402_1005Metric"
+		(property "Footprint" "Diode_SMD:D_0805_2012Metric"
 			(at 397.51 166.37 0)
 			(effects
@@
 			)
 		)
-		(property "Footprint" "Diode_SMD:D_0402_1005Metric"
+		(property "Footprint" "Diode_SMD:D_0805_2012Metric"
 			(at 370.84 180.34 0)
 			(effects
@@
 			)
 		)
-		(property "Footprint" "Diode_SMD:D_0402_1005Metric"
+		(property "Footprint" "Diode_SMD:D_MicroMELF"
 			(at 370.84 177.8 0)
 			(effects
@@
 			)
 		)
-		(property "Footprint" "Diode_SMD:D_0402_1005Metric"
+		(property "Footprint" "Diode_SMD:D_MicroMELF"
 			(at 369.57 127 0)
 			(effects
@@
 			)
 		)
-		(property "Footprint" "Diode_SMD:D_0402_1005Metric"
+		(property "Footprint" "Diode_SMD:D_0805_2012Metric"
 			(at 397.51 128.27 0)
 			(effects
@@
 			)
 		)
-		(property "Footprint" "Diode_SMD:D_0402_1005Metric"
+		(property "Footprint" "Diode_SMD:D_0805_2012Metric"
 			(at 397.51 146.05 0)
 			(effects
@@
 			)
 		)
-		(property "Footprint" "Diode_SMD:D_0402_1005Metric"
+		(property "Footprint" "Diode_SMD:D_0805_2012Metric"
 			(at 397.51 163.83 0)
 			(effects
@@
 			)
 		)
-		(property "Footprint" "Diode_SMD:D_0402_1005Metric"
+		(property "Footprint" "Diode_SMD:D_MicroMELF"
 			(at 369.57 139.7 0)
 			(effects
@@
 			)
 		)
-		(property "Footprint" "Diode_SMD:D_0402_1005Metric"
+		(property "Footprint" "Diode_SMD:D_0805_2012Metric"
 			(at 397.51 140.97 0)
 			(effects
@@
 			)
 		)
-		(property "Footprint" "Diode_SMD:D_0402_1005Metric"
+		(property "Footprint" "Diode_SMD:D_0805_2012Metric"
 			(at 369.57 152.4 0)
 			(effects
@@
 			)
 		)
-		(property "Footprint" "Diode_SMD:D_0402_1005Metric"
+		(property "Footprint" "Diode_SMD:D_0805_2012Metric"
 			(at 397.51 125.73 0)
 			(effects
@@
 			)
 		)
-		(property "Footprint" "Diode_SMD:D_0402_1005Metric"
+		(property "Footprint" "Diode_SMD:D_0805_2012Metric"
 			(at 397.51 171.45 0)
 			(effects
@@
 			)
 		)
-		(property "Footprint" "Diode_SMD:D_0402_1005Metric"
+		(property "Footprint" "Diode_SMD:D_MicroMELF"
 			(at 370.84 209.55 0)
 			(effects
@@
 			)
 		)
-		(property "Footprint" "Diode_SMD:D_0402_1005Metric"
+		(property "Footprint" "Diode_SMD:D_0805_2012Metric"
 			(at 397.51 156.21 0)
 			(effects
@@
 			)
 		)
-		(property "Footprint" "Diode_SMD:D_0402_1005Metric"
+		(property "Footprint" "Diode_SMD:D_MicroMELF"
 			(at 370.84 172.72 0)
 			(effects
@@
 			)
 		)
-		(property "Footprint" "Diode_SMD:D_0402_1005Metric"
+		(property "Footprint" "Diode_SMD:D_0805_2012Metric"
 			(at 369.57 107.95 0)
 			(effects
@@
 			)
 		)
-		(property "Footprint" "Diode_SMD:D_0402_1005Metric"
+		(property "Footprint" "Diode_SMD:D_0805_2012Metric"
 			(at 397.51 173.99 0)
 			(effects
@@
 			)
 		)
-		(property "Footprint" "Diode_SMD:D_0402_1005Metric"
+		(property "Footprint" "Diode_SMD:D_0805_2012Metric"
 			(at 397.51 148.59 0)
 			(effects
@@
 			)
 		)
-		(property "Footprint" "Diode_SMD:D_0402_1005Metric"
+		(property "Footprint" "Diode_SMD:D_0805_2012Metric"
 			(at 397.51 153.67 0)
 			(effects
@@
 			)
 		)
-		(property "Footprint" "Diode_SMD:D_0402_1005Metric"
+		(property "Footprint" "Diode_SMD:D_0805_2012Metric"
 			(at 397.51 113.03 0)
 			(effects
@@
 			)
 		)
-		(property "Footprint" "Diode_SMD:D_0402_1005Metric"
+		(property "Footprint" "Diode_SMD:D_0805_2012Metric"
 			(at 397.51 158.75 0)
 			(effects
@@
 			)
 		)
-		(property "Footprint" "Diode_SMD:D_0402_1005Metric"
+		(property "Footprint" "Diode_SMD:D_MicroMELF"
 			(at 370.84 212.09 0)
 			(effects
@@
 			)
 		)
-		(property "Footprint" "Diode_SMD:D_0402_1005Metric"
+		(property "Footprint" "Diode_SMD:D_0805_2012Metric"
 			(at 397.51 184.15 0)
 			(effects
@@
 			)
 		)
-		(property "Footprint" "Diode_SMD:D_0402_1005Metric"
+		(property "Footprint" "Diode_SMD:D_0805_2012Metric"
 			(at 397.51 135.89 0)
 			(effects
@@
 			)
 		)
-		(property "Footprint" "Diode_SMD:D_0402_1005Metric"
+		(property "Footprint" "Diode_SMD:D_MicroMELF"
 			(at 369.57 133.35 0)
 			(effects
@@
 			)
 		)
-		(property "Footprint" "Diode_SMD:D_0402_1005Metric"
+		(property "Footprint" "Diode_SMD:D_0805_2012Metric"
 			(at 397.51 186.69 0)
 			(effects
@@
 			)
 		)
-		(property "Footprint" "Diode_SMD:D_0402_1005Metric"
+		(property "Footprint" "Diode_SMD:D_0805_2012Metric"
 			(at 397.51 110.49 0)
 			(effects
@@
 			)
 		)
-		(property "Footprint" "Diode_SMD:D_0402_1005Metric"
+		(property "Footprint" "Diode_SMD:D_0805_2012Metric"
 			(at 397.51 151.13 0)
 			(effects
@@
 			)
 		)
-		(property "Footprint" "Diode_SMD:D_0402_1005Metric"
+		(property "Footprint" "Diode_SMD:D_0805_2012Metric"
 			(at 397.51 115.57 0)
 			(effects
@@
 			)
 		)
-		(property "Footprint" "Diode_SMD:D_0402_1005Metric"
+		(property "Footprint" "Diode_SMD:D_0805_2012Metric"
 			(at 397.51 133.35 0)
 			(effects
@@
 			)
 		)
-		(property "Footprint" "Diode_SMD:D_0402_1005Metric"
+		(property "Footprint" "Diode_SMD:D_0805_2012Metric"
 			(at 369.57 114.3 0)
 			(effects
@@
 			)
 		)
-		(property "Footprint" "Diode_SMD:D_0402_1005Metric"
+		(property "Footprint" "Diode_SMD:D_0805_2012Metric"
 			(at 397.51 118.11 0)
 			(effects
@@
 			)
 		)
-		(property "Footprint" "Diode_SMD:D_0402_1005Metric"
+		(property "Footprint" "Diode_SMD:D_0805_2012Metric"
 			(at 397.51 176.53 0)
 			(effects
@@
 			)
 		)
-		(property "Footprint" "Diode_SMD:D_0402_1005Metric"
+		(property "Footprint" "Diode_SMD:D_MicroMELF"
 			(at 370.84 193.04 0)
 			(effects
@@
 			)
 		)
-		(property "Footprint" "Diode_SMD:D_0402_1005Metric"
+		(property "Footprint" "Diode_SMD:D_MicroMELF"
 			(at 370.84 187.96 0)
 			(effects
@@
 			)
 		)
-		(property "Footprint" "Diode_SMD:D_0402_1005Metric"
+		(property "Footprint" "Diode_SMD:D_0805_2012Metric"
 			(at 397.51 168.91 0)
 			(effects
@@
 			)
 		)
-		(property "Footprint" "Diode_SMD:D_0402_1005Metric"
+		(property "Footprint" "Diode_SMD:D_0805_2012Metric"
 			(at 397.51 161.29 0)
 			(effects
@@
 			)
 		)
-		(property "Footprint" "Diode_SMD:D_0402_1005Metric"
+		(property "Footprint" "Diode_SMD:D_MicroMELF"
 			(at 370.84 167.64 0)
 			(effects
@@
 			)
 		)
-		(property "Footprint" "Diode_SMD:D_0402_1005Metric"
+		(property "Footprint" "Diode_SMD:D_MicroMELF"
 			(at 369.57 120.65 0)
 			(effects
@@
 			)
 		)
-		(property "Footprint" "Diode_SMD:D_0402_1005Metric"
+		(property "Footprint" "Diode_SMD:D_0805_2012Metric"
 			(at 397.51 120.65 0)
 			(effects
@@
 			)
 		)
-		(property "Footprint" "Diode_SMD:D_0402_1005Metric"
+		(property "Footprint" "Diode_SMD:D_0805_2012Metric"
 			(at 397.51 138.43 0)
 			(effects
@@
 			)
 		)
-		(property "Footprint" "Diode_SMD:D_0402_1005Metric"
+		(property "Footprint" "Diode_SMD:D_0805_2012Metric"
 			(at 397.51 143.51 0)
 			(effects
@@
 			)
 		)
-		(property "Footprint" "Diode_SMD:D_0402_1005Metric"
+		(property "Footprint" "Diode_SMD:D_0805_2012Metric"
 			(at 397.51 130.81 0)
 			(effects
@@
 			)
 		)
-		(property "Footprint" "Diode_SMD:D_0402_1005Metric"
+		(property "Footprint" "Diode_SMD:D_MicroMELF"
 			(at 370.84 205.74 0)
 			(effects
@@
 			)
 		)
-		(property "Footprint" "Diode_SMD:D_0402_1005Metric"
+		(property "Footprint" "Diode_SMD:D_0805_2012Metric"
 			(at 397.51 181.61 0)
 			(effects
@@
 			)
 		)
-		(property "Footprint" "Diode_SMD:D_0402_1005Metric"
+		(property "Footprint" "Diode_SMD:D_MicroMELF"
 			(at 370.84 182.88 0)
 			(effects
@@
 			)
 		)
-		(property "Footprint" "Diode_SMD:D_0402_1005Metric"
+		(property "Footprint" "Diode_SMD:D_MicroMELF"
 			(at 370.84 170.18 0)
 			(effects
