File: pcb/kicad/POWER_SHEET.kicad_sch (KiCad schematic)
At the start: 10 parts, among them J1 USB_B_Micro, U1 LMS1585AIS-3.3

Commit message: Add test points to schematic and pcb
- Test points are in the form of a 0402 (Imperial) diode footprint with
  pin 1 denoting the signal being tested and pin 2 always being GND
- Therefore the silkscreen GND has been omitted, follow the signal name
  to the "." which denotes pin 1
- 0402 package is intended for a oscilloscope probe with the ground
  probe tip for a low impedance path to ground
- ARM SWD test points can be via the hook clip along with a clip to
  ground nearby, as the SWD is a THT footprint I didn't feel the need to
  again expose out more pins for a SMD based test point
- Since the pads for the I2S mic are already exposed, it seemed
  counterintuitive to then make additional test points for the I2S
  pads. The silkscreen describes the pinout such that on-the-fly test
  points can be used in conjunction with nearby ground vias and pads
Parts:
- added TP1, TP2, TP3: TestPoint_2Pole, Diode_SMD:D_0402_1005Metric, symbol Connector:TestPoint_2Pole
Connections:
- net +3V3: now also TP3.1
- net +5V: now also TP2.1
- net GND: now also TP1.2, TP2.2, TP3.2
- net VBUS: now also TP1.1

Commit message: Update bom/mpn attributes
Parts:
- C1: MPN (none) -> GCM188R71H103KA37J
- C2: MPN (none) -> C0603C104J3RACTU
- C3, C4: MPN (none) -> EDH106M016A9BAA
- D2: value LED_Small_Filled -> 3V3 LED (RED); MPN (none) -> LTST-C190KRKT
- FB1: value 30R @ 100 MHz -> 300R @ 100 MHz; MPN (none) -> HI2220R301R-10
- TP1, TP2, TP3: now left out of the parts list
Changed lines of the file:
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@@
 		(unit 1)
 		(exclude_from_sim no)
-		(in_bom yes)
+		(in_bom no)
 		(on_board yes)
 		(dnp no)
@@
 			)
 		)
+		(property "MPN" "EDH106M016A9BAA"
+			(at 113.03 60.96 0)
+			(effects
+				(font
+					(size 1.27 1.27)
+				)
+				(hide yes)
+			)
+		)
 		(pin "1"
 		)
@@
 			)
 		)
-		(property "Value" "LED_Small_Filled"
+		(property "Value" "3V3 LED (RED)"
 			(at 184.0865 50.8 0)
 			(effects
@@
 		)
 		(property "Sim.Pins" "1=K 2=A"
+			(at 184.15 54.61 0)
+			(effects
+				(font
+					(size 1.27 1.27)
+				)
+				(hide yes)
+			)
+		)
+		(property "MPN" "LTST-C190KRKT"
 			(at 184.15 54.61 0)
 			(effects
@@
 			)
 		)
-		(property "Value" "30R @ 100 MHz"
+		(property "Value" "300R @ 100 MHz"
 			(at 91.3892 49.53 90)
 			(effects
@@
 			)
 		)
+		(property "MPN" "HI2220R301R-10"
+			(at 91.44 54.61 90)
+			(effects
+				(font
+					(size 1.27 1.27)
+				)
+				(hide yes)
+			)
+		)
 		(pin "2"
 		)
@@
 			)
 		)
+		(property "MPN" "C0603C104J3RACTU"
+			(at 100.33 60.96 0)
+			(effects
+				(font
+					(size 1.27 1.27)
+				)
+				(hide yes)
+			)
+		)
 		(pin "1"
 		)
@@
 		(unit 1)
 		(exclude_from_sim no)
-		(in_bom yes)
+		(in_bom no)
 		(on_board yes)
 		(dnp no)
@@
 			)
 		)
+		(property "MPN" "EDH106M016A9BAA"
+			(at 177.8 62.23 0)
+			(effects
+				(font
+					(size 1.27 1.27)
+				)
+				(hide yes)
+			)
+		)
 		(pin "1"
 		)
@@
 			)
 		)
+		(property "MPN" "GCM188R71H103KA37J"
+			(at 81.28 60.96 0)
+			(effects
+				(font
+					(size 1.27 1.27)
+				)
+				(hide yes)
+			)
+		)
 		(pin "1"
 		)
@@
 		(unit 1)
 		(exclude_from_sim no)
-		(in_bom yes)
-		(on_board yes)
-		(dnp no)
+		(in_bom no)
+		(on_board yes)
+		(dnp no)

Commit message: Replace test point footprints
- Quite difficult to probe the 0402 SMD sized test points with my PCBite
  probes
- End up scraping up the PCB trying to probe my test points as the gap
  is too small (on the 0402 footprint)
- The 0805 and microMELF footprints are appropriately sized for hands
  free probing
- Used microMELF footprints where space was very tight (as the microMELF
  occupies a slightly smaller area)
Parts:
- TP1, TP3: footprint Diode_SMD:D_0402_1005Metric -> Diode_SMD:D_MicroMELF
- TP2: footprint Diode_SMD:D_0402_1005Metric -> Diode_SMD:D_0805_2012Metric
Changed lines of the file:
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@@
 			)
 		)
-		(property "Footprint" "Diode_SMD:D_0402_1005Metric"
+		(property "Footprint" "Diode_SMD:D_0805_2012Metric"
 			(at 44.45 111.76 0)
 			(effects
@@
 			)
 		)
-		(property "Footprint" "Diode_SMD:D_0402_1005Metric"
+		(property "Footprint" "Diode_SMD:D_MicroMELF"
 			(at 44.45 119.38 0)
 			(effects
@@
 			)
 		)
-		(property "Footprint" "Diode_SMD:D_0402_1005Metric"
+		(property "Footprint" "Diode_SMD:D_MicroMELF"
 			(at 44.45 104.14 0)
 			(effects
