File: pcb/kicad/I2S_MIC.kicad_sch (KiCad schematic)
At the start: 4 parts

Commit message: Update parts/mpns/descriptions etc.
- Incorrect LED part, was 0805 package instead of 0603
- Added MPNs for other parts (mostly ones I already own multiples of)
- Update schematics?
Parts:
- MK1: MPN (none) -> MSM261S4030H0R
Changed lines of the file:
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@@
+			)
+		)
+		(property "MPN" "MSM261S4030H0R"
+			(at 83.82 54.61 0)
+			(effects
+				(font
+					(size 1.27 1.27)
+				)
+				(hide yes)
 			)
 		)

Commit message: Update capcitor annotations
- One less capacitor therefore the symbol annotations need to be changed
Parts:
- renumbered C6 to C5, C7 to C6
Changed lines of the file:
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@@
 	(title_block
 		(title "I2S Mic")
-		(date "2024-11-18")
-		(rev "v01")
+		(date "2025-05-21")
+		(rev "v02")
 		(comment 4 "Same as Fermion I2S mic breakout board")
 	)
@@
 		(on_board yes)
 		(dnp no)
-		(property "Reference" "C7"
+		(property "Reference" "C6"
 			(at 134.62 52.07 90)
 			(effects
@@
 			(project ""
 				(path "/e164be4c-4870-49b4-a08f-d162a756edc1/caff8704-a6ad-414b-a861-33b9c55688a3"
-					(reference "C7")
+					(reference "C6")
 					(unit 1)
 				)
@@
 		(dnp no)
 		(fields_autoplaced yes)
-		(property "Reference" "C6"
+		(property "Reference" "C5"
 			(at 134.62 33.02 90)
 			(effects
@@
 			(project "i2s_spekky_matrix"
 				(path "/e164be4c-4870-49b4-a08f-d162a756edc1/caff8704-a6ad-414b-a861-33b9c55688a3"
-					(reference "C6")
+					(reference "C5")
 					(unit 1)
 				)

Commit message: Update pcb footprint for i2s mic
Parts:
- MK1: footprint spekky_matrix:LGA-8_2x4_3.0x4.0mm_P1.0mm -> spekky_matrix:LGA-8_2x4_3.0x4.0mm_P1.0mm_Hand_Solder
Changed lines of the file:
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@@
 			)
 		)
-		(property "Footprint" "spekky_matrix:LGA-8_2x4_3.0x4.0mm_P1.0mm"
+		(property "Footprint" "spekky_matrix:LGA-8_2x4_3.0x4.0mm_P1.0mm_Hand_Solder"
 			(at 83.82 54.61 0)
 			(effects

Commit message: Update bom/mpn attributes
Parts:
- C5: MPN (none) -> C1608X5R1A106K080AC
- C6: MPN (none) -> C0603C104J3RACTU
- R2: MPN (none) -> H4P100KDZA
Changed lines of the file:
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@@
+			)
+		)
+		(property "MPN" "C0603C104J3RACTU"
+			(at 134.62 48.26 90)
+			(effects
+				(font
+					(size 1.27 1.27)
+				)
+				(hide yes)
 			)
 		)
@@
 			)
 		)
+		(property "MPN" "H4P100KDZA"
+			(at 125.73 69.85 0)
+			(effects
+				(font
+					(size 1.27 1.27)
+				)
+				(hide yes)
+			)
+		)
 		(pin "1"
 		)
@@
 			(effects
 				(font
+					(size 1.27 1.27)
+				)
+				(hide yes)
+			)
+		)
+		(property "MPN" "C1608X5R1A106K080AC"
+			(at 134.62 40.64 90)
+			(effects
+				(font

Commit message: Correct 100k resistor part number
- Previous was a THT component, corrected to SMD 0603 imperial
Parts:
- R2: MPN H4P100KDZA -> RP73PF1J100KBTDF
Changed lines of the file:
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@@
 			)
 		)
-		(property "MPN" "H4P100KDZA"
+		(property "MPN" "RP73PF1J100KBTDF"
 			(at 125.73 69.85 0)
 			(effects

Commit message: Add test point for i2s sck pin
- Probing in the I2S pins directly is challenging for adjacent pins
- Exposing the SCK pad as it's adjacent to the GND pin and would benefit
  from a test point
- Updated schematic revisions where necessary
Parts:
- added TP60: TestPoint_2Pole, Diode_SMD:D_MicroMELF, symbol Connector:TestPoint_2Pole
Connections:
- net GND: now also TP60.2
- net I2S_SCK: now also TP60.1
Changed lines of the file:
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@@
 	(title_block
 		(title "I2S Mic")
-		(date "2025-05-21")
-		(rev "v02")
+		(date "2026-01-04")
+		(rev "v03")
 		(comment 4 "Same as Fermion I2S mic breakout board")
 	)
@@
 	(wire
 		(pts
+			(xy 172.72 63.5) (xy 172.72 66.04)
+		)
+		(stroke
+			(width 0)
+			(type default)
+		)
+	)
+	(wire
+		(pts
 			(xy 105.41 58.42) (xy 121.92 58.42)
 		)
@@
 	(wire
 		(pts
+			(xy 156.21 63.5) (xy 158.75 63.5)
+		)
+		(stroke
+			(width 0)
+			(type default)
+		)
+	)
+	(wire
+		(pts
 			(xy 67.31 53.34) (xy 67.31 66.04)
 		)
@@
 		(pts
 			(xy 121.92 40.64) (xy 121.92 48.26)
+		)
+		(stroke
+			(width 0)
+			(type default)
+		)
+	)
+	(wire
+		(pts
+			(xy 168.91 63.5) (xy 172.72 63.5)
 		)
 		(stroke
@@
 			)
 			(justify left)
+		)
+	)
+	(hierarchical_label "I2S_SCK"
+		(shape input)
+		(at 156.21 63.5 180)
+		(effects
+			(font
+				(size 1.27 1.27)
+			)
+			(justify right)
 		)
 	)
@@
 				(path "/e164be4c-4870-49b4-a08f-d162a756edc1/caff8704-a6ad-414b-a861-33b9c55688a3"
 					(reference "#PWR015")
+					(unit 1)
+				)
+			)
+		)
+	)
+	(symbol
+		(lib_id "power:GNDREF")
+		(at 172.72 66.04 0)
+		(unit 1)
+		(exclude_from_sim no)
+		(in_bom yes)
+		(on_board yes)
+		(dnp no)
+		(property "Reference" "#PWR062"
+			(at 172.72 72.39 0)
+			(effects
+				(font
+					(size 1.27 1.27)
+				)
+				(hide yes)
+			)
+		)
+		(property "Value" "GND"
+			(at 172.72 69.85 0)
+			(effects
+				(font
+					(size 1.27 1.27)
+				)
+				(hide yes)
+			)
+		)
+		(property "Footprint" ""
+			(at 172.72 66.04 0)
+			(effects
+				(font
+					(size 1.27 1.27)
+				)
+				(hide yes)
+			)
+		)
+		(property "Datasheet" ""
+			(at 172.72 66.04 0)
+			(effects
+				(font
+					(size 1.27 1.27)
+				)
+				(hide yes)
+			)
+		)
+		(property "Description" "Power symbol creates a global label with name \"GND\" , reference supply ground"
+			(at 172.72 66.04 0)
+			(effects
+				(font
+					(size 1.27 1.27)
+				)
+				(hide yes)
+			)
+		)
+		(pin "1"
+		)
+		(instances
+			(project "spekky_matrix"
+				(path "/e164be4c-4870-49b4-a08f-d162a756edc1/caff8704-a6ad-414b-a861-33b9c55688a3"
+					(reference "#PWR062")
 					(unit 1)
 				)
@@
 					(unit 1)
 				)
+			)
+		)
+	)
+	(symbol
+		(lib_id "Connector:TestPoint_2Pole")
+		(at 163.83 63.5 0)
+		(unit 1)
+		(exclude_from_sim no)
+		(in_bom no)
+		(on_board yes)
+		(dnp no)
+		(property "Reference" "TP60"
+			(at 163.83 61.722 0)
+			(effects
+				(font
+					(size 1.27 1.27)
+				)
+			)
+		)
+		(property "Value" "TestPoint_2Pole"
+			(at 163.83 60.96 0)
+			(effects
+				(font
+					(size 1.27 1.27)
+				)
+				(hide yes)
+			)
+		)
+		(property "Footprint" "Diode_SMD:D_MicroMELF"
+			(at 163.83 63.5 0)
+			(effects
+				(font
+					(size 1.27 1.27)
+				)
+				(hide yes)
+			)
+		)
+		(property "Datasheet" "~"
+			(at 163.83 63.5 0)
+			(effects
+				(font
+					(size 1.27 1.27)
+				)
+				(hide yes)
+			)
+		)
+		(property "Description" "2-polar test point"
+			(at 163.83 63.5 0)
+			(effects
+				(font
+					(size 1.27 1.27)
+				)
+				(hide yes)
+			)
+		)
+		(pin "2"
+		)
+		(pin "1"
+		)
+		(instances
+			(project "spekky_matrix"
+				(path "/e164be4c-4870-49b4-a08f-d162a756edc1/caff8704-a6ad-414b-a861-33b9c55688a3"
+					(reference "TP60")
+					(unit 1)
+				)

Commit message: Add comment for i2s test points
- No test points needed for SD and WS as there is a GND pin 2 pins away
  which the PCBite probes can be used handsfree in this case
Other:
- note added: "Can probe the SD and WS pins directly (PCBite works handsfree when the GND pin is 2 pins away)"
Changed lines of the file:
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@@
 		(comment 4 "Same as Fermion I2S mic breakout board")
+	)
+	(text "Can probe the SD and WS pins directly\n(PCBite works handsfree when the GND pin\nis 2 pins away)"
+		(exclude_from_sim no)
+		(at 164.084 75.184 0)
+		(effects
+			(font
+				(size 1.27 1.27)
+			)
+		)
 	)
 	(junction
